File: Tarea 3/Diseño PCB/PLC4UNI/PLC4UNI.kicad_sch (KiCad schematic)
At the start: 2 parts, among them J1 Screw_Terminal_01x09, J2 Screw_Terminal_01x18

Commit message: Tarea 3
Parts:
- removed J1: Screw_Terminal_01x09, TerminalBlock:TerminalBlock_MaiXu_MX126-5.0-09P_1x09_P5.00mm, symbol Connector:Screw_Terminal_01x09
- removed J2: Screw_Terminal_01x18, TerminalBlock:TerminalBlock_MaiXu_MX126-5.0-18P_1x18_P5.00mm, symbol Connector:Screw_Terminal_01x18
- added J1: Screw_Terminal_01x03, TerminalBlock:TerminalBlock_MaiXu_MX126-5.0-03P_1x03_P5.00mm, symbol Connector:Screw_Terminal_01x03
Connections:
- new net Board-PLC4UNI-G1w/con_RS485_A: J1.1 (Pin_1)
- new net Board-PLC4UNI-G1w/con_RS485_B: J1.2 (Pin_2)
- new net GNDPWR: J1.3 (Pin_3)
Other:
- added sheet Board-PLC4UNI-G1w (Board-PLC4UNI-G1w.kicad_sch)
Changed lines of the file:
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@@
 	(generator_version "9.0")
 	(paper "A4")
+	(wire
+		(pts
+			(xy 154.94 93.98) (xy 154.94 97.79)
+		)
+		(stroke
+			(width 0)
+			(type default)
+		)
+	)
+	(wire
+		(pts
+			(xy 148.59 91.44) (xy 154.94 91.44)
+		)
+		(stroke
+			(width 0)
+			(type default)
+		)
+	)
+	(wire
+		(pts
+			(xy 148.59 88.9) (xy 154.94 88.9)
+		)
+		(stroke
+			(width 0)
+			(type default)
+		)
+	)
 	(symbol
-		(lib_id "Connector:Screw_Terminal_01x18")
-		(at 146.05 105.41 0)
-		(unit 1)
-		(exclude_from_sim no)
-		(in_bom yes)
-		(on_board yes)
-		(dnp no)
-		(fields_autoplaced yes)
-		(property "Reference" "J2"
-			(at 148.59 105.4099 0)
-			(effects
-				(font
-					(size 1.27 1.27)
-				)
-				(justify left)
-			)
-		)
-		(property "Value" "Screw_Terminal_01x18"
-			(at 148.59 107.9499 0)
-			(effects
-				(font
-					(size 1.27 1.27)
-				)
-				(justify left)
-			)
-		)
-		(property "Footprint" "TerminalBlock:TerminalBlock_MaiXu_MX126-5.0-18P_1x18_P5.00mm"
-			(at 146.05 105.41 0)
-			(effects
-				(font
-					(size 1.27 1.27)
-				)
-				(hide yes)
-			)
-		)
-		(property "Datasheet" "~"
-			(at 146.05 105.41 0)
-			(effects
-				(font
-					(size 1.27 1.27)
-				)
-				(hide yes)
-			)
-		)
-		(property "Description" "Generic screw terminal, single row, 01x18, script generated (kicad-library-utils/schlib/autogen/connector/)"
-			(at 146.05 105.41 0)
-			(effects
-				(font
-					(size 1.27 1.27)
-				)
-				(hide yes)
-			)
-		)
-		(pin "2"
-		)
-		(pin "3"
-		)
-		(pin "14"
-		)
-		(pin "18"
-		)
-		(pin "12"
-		)
-		(pin "16"
-		)
-		(pin "6"
-		)
-		(pin "13"
-		)
-		(pin "15"
-		)
-		(pin "17"
-		)
-		(pin "4"
-		)
-		(pin "7"
-		)
-		(pin "5"
-		)
-		(pin "8"
-		)
-		(pin "9"
-		)
-		(pin "1"
-		)
-		(pin "11"
-		)
-		(pin "10"
-		)
-		(instances
-			(project ""
-				(path "/acad40d5-ac6b-4a60-8788-299f56574d0c"
-					(reference "J2")
-					(unit 1)
-				)
-			)
-		)
-	)
-	(symbol
-		(lib_id "Connector:Screw_Terminal_01x09")
-		(at 107.95 97.79 0)
+		(lib_id "Connector:Screw_Terminal_01x03")
+		(at 160.02 91.44 0)
 		(unit 1)
 		(exclude_from_sim no)
@@
 		(fields_autoplaced yes)
 		(property "Reference" "J1"
-			(at 110.49 96.5199 0)
+			(at 162.56 90.1699 0)
 			(effects
 				(font
@@
 			)
 		)
-		(property "Value" "Screw_Terminal_01x09"
-			(at 110.49 99.0599 0)
+		(property "Value" "Screw_Terminal_01x03"
+			(at 162.56 92.7099 0)
 			(effects
 				(font
@@
 			)
 		)
-		(property "Footprint" "TerminalBlock:TerminalBlock_MaiXu_MX126-5.0-09P_1x09_P5.00mm"
-			(at 107.95 97.79 0)
+		(property "Footprint" "TerminalBlock:TerminalBlock_MaiXu_MX126-5.0-03P_1x03_P5.00mm"
+			(at 160.02 91.44 0)
 			(effects
 				(font
@@
 		)
 		(property "Datasheet" "~"
-			(at 107.95 97.79 0)
-			(effects
-				(font
-					(size 1.27 1.27)
-				)
-				(hide yes)
-			)
-		)
-		(property "Description" "Generic screw terminal, single row, 01x09, script generated (kicad-library-utils/schlib/autogen/connector/)"
-			(at 107.95 97.79 0)
-			(effects
-				(font
-					(size 1.27 1.27)
-				)
-				(hide yes)
-			)
+			(at 160.02 91.44 0)
+			(effects
+				(font
+					(size 1.27 1.27)
+				)
+				(hide yes)
+			)
+		)
+		(property "Description" "Generic screw terminal, single row, 01x03, script generated (kicad-library-utils/schlib/autogen/connector/)"
+			(at 160.02 91.44 0)
+			(effects
+				(font
+					(size 1.27 1.27)
+				)
+				(hide yes)
+			)
+		)
+		(property "Part Number" "KANGNEX WJ128V-5.0-3P"
+			(at 160.02 91.44 0)
+			(effects
+				(font
+					(size 1.27 1.27)
+				)
+				(hide yes)
+			)
+		)
+		(pin "2"
 		)
 		(pin "3"
 		)
-		(pin "8"
-		)
 		(pin "1"
-		)
-		(pin "6"
-		)
-		(pin "7"
-		)
-		(pin "9"
-		)
-		(pin "5"
-		)
-		(pin "2"
-		)
-		(pin "4"
 		)
 		(instances
@@
 				)
 			)
+		)
+	)
+	(symbol
+		(lib_id "power:GNDPWR")
+		(at 154.94 97.79 0)
+		(unit 1)
+		(exclude_from_sim no)
+		(in_bom yes)
+		(on_board yes)
+		(dnp no)
+		(fields_autoplaced yes)
+		(property "Reference" "#PWR01"
+			(at 154.94 102.87 0)
+			(effects
+				(font
+					(size 1.27 1.27)
+				)
+				(hide yes)
+			)
+		)
+		(property "Value" "GNDPWR"
+			(at 154.813 101.6 0)
+			(effects
+				(font
+					(size 1.27 1.27)
+				)
+			)
+		)
+		(property "Footprint" ""
+			(at 154.94 99.06 0)
+			(effects
+				(font
+					(size 1.27 1.27)
+				)
+				(hide yes)
+			)
+		)
+		(property "Datasheet" ""
+			(at 154.94 99.06 0)
+			(effects
+				(font
+					(size 1.27 1.27)
+				)
+				(hide yes)
+			)
+		)
+		(property "Description" "Power symbol creates a global label with name \"GNDPWR\" , global ground"
+			(at 154.94 97.79 0)
+			(effects
+				(font
+					(size 1.27 1.27)
+				)
+				(hide yes)
+			)
+		)
+		(pin "1"
+		)
+		(instances
+			(project ""
+				(path "/acad40d5-ac6b-4a60-8788-299f56574d0c"
+					(reference "#PWR01")
+					(unit 1)
+				)
+			)
+		)
+	)
+	(sheet
+		(at 96.52 74.93)
+		(size 52.07 34.29)
+		(exclude_from_sim no)
+		(in_bom yes)
+		(on_board yes)
+		(dnp no)
+		(fields_autoplaced yes)
+		(stroke
+			(width 0.1524)
+			(type solid)
+		)
+		(fill
+			(color 0 0 0 0.0000)
+		)
+		(property "Sheetname" "Board-PLC4UNI-G1w"
+			(at 96.52 74.2184 0)
+			(effects
+				(font
+					(size 1.27 1.27)
+				)
+				(justify left bottom)
+			)
+		)
+		(property "Sheetfile" "Board-PLC4UNI-G1w.kicad_sch"
+			(at 96.52 109.8046 0)
+			(effects
+				(font
+					(size 1.27 1.27)
+				)
+				(justify left top)
+			)
+		)
+		(pin "con_RS485_A" bidirectional
+			(at 148.59 88.9 0)
+			(effects
+				(font
+					(size 1.27 1.27)
+				)
+				(justify right)
+			)
+		)
+		(pin "con_RS485_B" bidirectional
+			(at 148.59 91.44 0)
+			(effects
+				(font
+					(size 1.27 1.27)
+				)
+				(justify right)
+			)
+		)
+		(instances
+			(project "PLC4UNI"
+				(path "/acad40d5-ac6b-4a60-8788-299f56574d0c"
+					(page "2")
+				)
+			)

Commit message: Tarea 3
Parts:
- removed J1: Screw_Terminal_01x03, TerminalBlock:TerminalBlock_MaiXu_MX126-5.0-03P_1x03_P5.00mm, symbol Connector:Screw_Terminal_01x03
- added J1, J2: Screw_Terminal_01x18, symbol Connector:Screw_Terminal_01x18
Connections:
- new net Board-PLC4UNI-G1w/1_NPN_IN: J2.1 (Pin_1)
- new net Board-PLC4UNI-G1w/1_NPN_OUT: J1.1 (Pin_1)
- new net Board-PLC4UNI-G1w/1_PNP_IN: J2.4 (Pin_4)
- new net Board-PLC4UNI-G1w/1_PNP_OUT: J1.4 (Pin_4)
- new net Board-PLC4UNI-G1w/2_NPN_IN: J2.2 (Pin_2)
- new net Board-PLC4UNI-G1w/2_NPN_OUT: J1.2 (Pin_2)
- new net Board-PLC4UNI-G1w/2_PNP_IN: J2.5 (Pin_5)
- new net Board-PLC4UNI-G1w/2_PNP_OUT: J1.5 (Pin_5)
- new net Board-PLC4UNI-G1w/3_NPN_IN: J2.3 (Pin_3)
- new net Board-PLC4UNI-G1w/3_NPN_OUT: J1.3 (Pin_3)
- new net Board-PLC4UNI-G1w/3_PNP_IN: J2.6 (Pin_6)
- new net Board-PLC4UNI-G1w/3_PNP_OUT: J1.6 (Pin_6)
- new net Board-PLC4UNI-G1w/COM_A_RLY: J2.7 (Pin_7)
- new net Board-PLC4UNI-G1w/COM_B_RLY: J2.8 (Pin_8)
- new net Board-PLC4UNI-G1w/NC_B_RLY: J2.11 (Pin_11)
- new net Board-PLC4UNI-G1w/NO_A_RLY: J2.9 (Pin_9)
- new net Board-PLC4UNI-G1w/NO_B_RLY: J2.10 (Pin_10)
- new net Board-PLC4UNI-G1w/RS485_A: J1.7 (Pin_7)
- new net Board-PLC4UNI-G1w/RS485_B: J1.8 (Pin_8)
Other:
- sheet Board-PLC4UNI-G1w ports: added 1_NPN_IN, 1_NPN_OUT, 1_PNP_IN, 1_PNP_OUT, 2_NPN_IN, 2_NPN_OUT, 2_PNP_IN, 2_PNP_OUT, 3_NPN_IN, 3_NPN_OUT, 3_PNP_IN, 3_PNP_OUT, COM_A_RLY, COM_B_RLY, NC_B_RLY, NO_A_RLY, NO_B_RLY, RS485_A, RS485_B; removed con_RS485_A, con_RS485_B
- note added: "INPUT"
- note added: "OUTPUT"

Commit message: Tarea 3
Connections:
- net Board-PLC4UNI-G1w/1_NPN_IN: now also J2.5 (Pin_5); no longer J2.1 (Pin_1)
- net Board-PLC4UNI-G1w/1_NPN_OUT: now also J1.15 (Pin_15); no longer J1.1 (Pin_1)
- net Board-PLC4UNI-G1w/1_PNP_IN: now also J2.10 (Pin_10); no longer J2.4 (Pin_4)
- net Board-PLC4UNI-G1w/2_NPN_IN: now also J2.6 (Pin_6); no longer J2.2 (Pin_2)
- net Board-PLC4UNI-G1w/2_NPN_OUT: now also J1.16 (Pin_16); no longer J1.2 (Pin_2)
- net Board-PLC4UNI-G1w/2_PNP_IN: now also J2.11 (Pin_11); no longer J2.5 (Pin_5)
- net Board-PLC4UNI-G1w/3_NPN_IN: now also J2.7 (Pin_7); no longer J2.3 (Pin_3)
- net Board-PLC4UNI-G1w/3_NPN_OUT: now also J1.17 (Pin_17); no longer J1.3 (Pin_3)
- net Board-PLC4UNI-G1w/3_PNP_IN: now also J2.12 (Pin_12); no longer J2.6 (Pin_6)
- net Board-PLC4UNI-G1w/COM_A_RLY: now also J1.10 (Pin_10); no longer J2.7 (Pin_7)
- net Board-PLC4UNI-G1w/COM_B_RLY: now also J1.8 (Pin_8); no longer J2.8 (Pin_8)
- net Board-PLC4UNI-G1w/NC_B_RLY: now also J1.9 (Pin_9); no longer J2.11 (Pin_11)
- net Board-PLC4UNI-G1w/NO_A_RLY: now also J1.11 (Pin_11); no longer J2.9 (Pin_9)
- net Board-PLC4UNI-G1w/NO_B_RLY: now also J1.7 (Pin_7); no longer J2.10 (Pin_10)
- net Board-PLC4UNI-G1w/RS485_A: now also J1.1 (Pin_1); no longer J1.7 (Pin_7)
- net Board-PLC4UNI-G1w/RS485_B: now also J1.2 (Pin_2); no longer J1.8 (Pin_8)
- net Board-PLC4UNI-G1w/4_PNP_IN: now reaches J2.13 (Pin_13)
- net GND2: now reaches J2.14 (Pin_14)
- net Board-PLC4UNI-G1w/4_20Output: now reaches J1.12 (Pin_12)
- net GND4: now reaches J1.13 (Pin_13)
- net Board-PLC4UNI-G1w/0-10V_OUTPUT: now reaches J1.14 (Pin_14)
- net Board-PLC4UNI-G1w/4_NPN_OUT: now reaches J1.18 (Pin_18)
- new net +24V: J2.1 (Pin_1)
- new net Board-PLC4UNI-G1w/0-10_Voltage_Input: J2.9 (Pin_9)
- new net Board-PLC4UNI-G1w/4-20mA_Input: J2.3 (Pin_3)
- new net Board-PLC4UNI-G1w/4_NPN_IN: J2.8 (Pin_8)
- new net GND: J2.2 (Pin_2)
- new net GND1: J2.4 (Pin_4)
- new net GND3: J1.3 (Pin_3)
Other:
- sheet Board-PLC4UNI-G1w ports: added 0-10V_OUTPUT, 0-10_Voltage_Input, 4-20mA_Input, 4_20Output, 4_NPN_IN, 4_NPN_OUT, 4_PNP_IN; removed none

Commit message: Tarea  3
Connections:
- net GND1 is gone; now on net GND: J2.4 (Pin_4)
- net GND2 is gone; now on net GND: J2.14 (Pin_14)
- net GND3 is gone; now on net GND: J1.3 (Pin_3)
- net GND4 is gone; now on net GND: J1.13 (Pin_13)
Other:
- moved on the sheet: J2

Commit message: Tarea 3
Parts:
- J1, J2: footprint (none) -> TerminalBlock:TerminalBlock_MaiXu_MX126-5.0-18P_1x18_P5.00mm
Changed lines of the file:
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@@
 			)
 		)
-		(property "Footprint" ""
+		(property "Footprint" "TerminalBlock:TerminalBlock_MaiXu_MX126-5.0-18P_1x18_P5.00mm"
 			(at 85.09 71.12 0)
 			(effects
@@
 			)
 		)
-		(property "Footprint" ""
+		(property "Footprint" "TerminalBlock:TerminalBlock_MaiXu_MX126-5.0-18P_1x18_P5.00mm"
 			(at 156.21 71.12 0)
 			(effects
