File: Tarea 3/Diseño PCB/PLC4UNI/PLC4UNI_CPU.kicad_sch (KiCad schematic)
At the start: 4 parts, among them U1 ESP32-S3-WROOM-1

Commit message: Tarea 3
Parts:
- added C5: C, symbol Device:C
- added R52: R_US, symbol Device:R_US
Connections:
- net GND: now also C5.1
- net VDD: now also R52.1
- net FROMESP_OUT_IN-PNP_A: now reaches U1.20 (IO12)
- net FROMESP_OUT_IN-PNP_B: now reaches U1.21 (IO13)
- net FROMESP_OUT_IN-PNP_C: now reaches U1.22 (IO14)
- net FROMESP_SCLK_C: now reaches U1.24 (IO47)
- net FROMESP_OUT_IN-NPN_A: now reaches U1.27 (IO0)
- net at U1.3 (EN): now also C5.2, R52.2
- net FROMESP_OUT_IN-NPN_C: now reaches U1.38 (IO2)
- net FROMESP_OUT_IN-NPN_B: now reaches U1.39 (IO1)
- net FROMESP_SEL_VOUT: now reaches U1.7 (IO7)
- net FROMESP_SDA_V: now reaches U1.8 (IO15)
- net FROMESP_SCLK_V: now reaches U1.9 (IO16)
- net micro_RS485_control renamed FROMESP_SDA_C
- net micro_RS485_rx renamed ESP32_UART_B
- net micro_RS485_tx renamed ESP32_UART_A

Commit message: Tarea 3
Connections:
- net FROMESP_IN_OUT-PNP_C: now reaches U1.16 (IO46)
- net FROMESP_IN_OUT-PNP_B: now reaches U1.26 (IO45)
- net FROMESP_IN_OUT-NPN_A: now reaches U1.32 (IO39)
- net FROMESP_IN_OUT-NPN_B: now reaches U1.33 (IO40)
- net FROMESP_IN_OUT-NPN_C: now reaches U1.34 (IO41)
- net FROMESP_IN_OUT-PNP_A: now reaches U1.35 (IO42)
Changed lines of the file:
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@@
+	(wire
+		(pts
+			(xy 156.21 96.52) (xy 165.1 96.52)
+		)
+		(stroke
+			(width 0)
+			(type default)
+		)
+	)
 	(wire
 		(pts
@@
 	(wire
 		(pts
+			(xy 156.21 101.6) (xy 165.1 101.6)
+		)
+		(stroke
+			(width 0)
+			(type default)
+		)
+	)
+	(wire
+		(pts
+			(xy 156.21 104.14) (xy 165.1 104.14)
+		)
+		(stroke
+			(width 0)
+			(type default)
+		)
+	)
+	(wire
+		(pts
 			(xy 114.3 78.74) (xy 125.73 78.74)
 		)
@@
 	(wire
 		(pts
+			(xy 156.21 109.22) (xy 165.1 109.22)
+		)
+		(stroke
+			(width 0)
+			(type default)
+		)
+	)
+	(wire
+		(pts
 			(xy 68.58 67.31) (xy 69.85 67.31)
 		)
@@
 	(wire
 		(pts
+			(xy 156.21 106.68) (xy 165.1 106.68)
+		)
+		(stroke
+			(width 0)
+			(type default)
+		)
+	)
+	(wire
+		(pts
 			(xy 156.21 78.74) (xy 161.29 78.74)
 		)
@@
 		(pts
 			(xy 120.65 66.04) (xy 124.46 66.04)
+		)
+		(stroke
+			(width 0)
+			(type default)
+		)
+	)
+	(wire
+		(pts
+			(xy 156.21 99.06) (xy 165.1 99.06)
 		)
 		(stroke
@@
 			)
 			(justify right)
+		)
+	)
+	(hierarchical_label "FROMESP_IN_OUT-NPN_B"
+		(shape input)
+		(at 165.1 99.06 0)
+		(effects
+			(font
+				(size 1.27 1.27)
+			)
+			(justify left)
 		)
 	)
@@
 		)
 	)
+	(hierarchical_label "FROMESP_IN_OUT-PNP_B"
+		(shape input)
+		(at 165.1 106.68 0)
+		(effects
+			(font
+				(size 1.27 1.27)
+			)
+			(justify left)
+		)
+	)
 	(hierarchical_label "FROMESP_OUT_IN-NPN_B"
 		(shape input)
@@
 		)
 	)
+	(hierarchical_label "FROMESP_IN_OUT-PNP_C"
+		(shape input)
+		(at 165.1 109.22 0)
+		(effects
+			(font
+				(size 1.27 1.27)
+			)
+			(justify left)
+		)
+	)
 	(hierarchical_label "FROMESP_SDA_C"
 		(shape input)
@@
 		)
 	)
+	(hierarchical_label "FROMESP_IN_OUT-NPN_C"
+		(shape input)
+		(at 165.1 101.6 0)
+		(effects
+			(font
+				(size 1.27 1.27)
+			)
+			(justify left)
+		)
+	)
 	(hierarchical_label "ESP32_UART_A"
 		(shape input)
@@
 		(effects
 			(font
+				(size 1.27 1.27)
+			)
+			(justify left)
+		)
+	)
+	(hierarchical_label "FROMESP_IN_OUT-NPN_A"
+		(shape input)
+		(at 165.1 96.52 0)
+		(effects
+			(font
+				(size 1.27 1.27)
+			)
+			(justify left)
+		)
+	)
+	(hierarchical_label "FROMESP_IN_OUT-PNP_A"
+		(shape input)
+		(at 165.1 104.14 0)
+		(effects
+			(font

Commit message: Tarea 3
Connections:
- net RLY_B_INR: now reaches U1.36 (RXD0)
- net RLY_A_INR: now reaches U1.37 (TXD0)
Changed lines of the file:
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@@
+	(wire
+		(pts
+			(xy 156.21 68.58) (xy 160.02 68.58)
+		)
+		(stroke
+			(width 0)
+			(type default)
+		)
+	)
+	(wire
+		(pts
+			(xy 156.21 71.12) (xy 160.02 71.12)
+		)
+		(stroke
+			(width 0)
+			(type default)
+		)
+	)
 	(wire
 		(pts
@@
 		)
 	)
+	(hierarchical_label "RLY_A_INR"
+		(shape bidirectional)
+		(at 160.02 68.58 0)
+		(effects
+			(font
+				(size 1.27 1.27)
+			)
+			(justify left)
+		)
+	)
 	(hierarchical_label "FROMESP_IN_OUT-NPN_C"
 		(shape input)
@@
 		(effects
 			(font
+				(size 1.27 1.27)
+			)
+			(justify left)
+		)
+	)
+	(hierarchical_label "RLY_B_INR"
+		(shape bidirectional)
+		(at 160.02 71.12 0)
+		(effects
+			(font

Commit message: Tarea 3
Connections:
- net FROMESP_SCLK_C is gone; now on net FROMESP_IN_OUT-PNP_C: U1.24 (IO47)
- net FROMESP_IN_OUT-PNP_A: now also U1.26 (IO45); no longer U1.35 (IO42)
- net FROMESP_IN_OUT-PNP_B: now also U1.16 (IO46); no longer U1.26 (IO45)
- net FROMESP_IN_OUT-PNP_C: no longer U1.16 (IO46)
- net FROMESP_OUT_IN-PNP_A: now also U1.19 (IO11); no longer U1.20 (IO12)
- net FROMESP_OUT_IN-PNP_B: now also U1.20 (IO12); no longer U1.21 (IO13)
- net FROMESP_OUT_IN-PNP_C: now also U1.21 (IO13); no longer U1.22 (IO14)
- net FROMESP_OUT_IN-NPN_D: now reaches U1.15 (IO3)
- net FROMESP_4-20mA_Input: now reaches U1.23 (IO21)
- net FROMESP_SCLK_V renamed FROMESP_SCLK
- net FROMESP_SDA_C renamed FROMESP_Voltage_Input
- net FROMESP_SDA_V renamed FROMESP_SDA
- new net FROMESP_IN_OUT-NPN_D: U1.35 (IO42)
- new net FROMESP_OUT_IN-PNP_D: U1.22 (IO14)

Commit message: Tarea  3
Parts:
- added R64, R65: 4.7k, Resistor_SMD:R_0603_1608Metric, symbol Device:R
Connections:
- net FROMESP_IN_OUT-NPN_A: now also U1.22 (IO14); no longer U1.32 (IO39)
- net FROMESP_IN_OUT-NPN_B: now also U1.21 (IO13); no longer U1.33 (IO40)
- net FROMESP_IN_OUT-NPN_C: now also U1.20 (IO12); no longer U1.34 (IO41)
- net FROMESP_IN_OUT-NPN_D: now also U1.19 (IO11); no longer U1.35 (IO42)
- net FROMESP_IN_OUT-PNP_A: now also U1.18 (IO10); no longer U1.26 (IO45)
- net FROMESP_IN_OUT-PNP_B: now also U1.17 (IO9); no longer U1.16 (IO46)
- net FROMESP_IN_OUT-PNP_C: now also U1.12 (IO8); no longer U1.24 (IO47)
- net FROMESP_OUT_IN-PNP_A: now also U1.4 (IO4); no longer U1.19 (IO11)
- net FROMESP_OUT_IN-PNP_B: now also U1.5 (IO5); no longer U1.20 (IO12)
- net FROMESP_OUT_IN-PNP_C: now also U1.6 (IO6); no longer U1.21 (IO13)
- net FROMESP_OUT_IN-PNP_D: now also U1.7 (IO7); no longer U1.22 (IO14)
- net FROMESP_SCLK: now also U1.28 (IO35), R64.2; no longer U1.9 (IO16)
- net FROMESP_SDA: now also U1.29 (IO36), R65.2; no longer U1.8 (IO15)
- net FROMESP_SEL_VOUT: now also U1.30 (IO37); no longer U1.7 (IO7)
- net FROMESP_Voltage_Input: now also U1.8 (IO15); no longer U1.25 (IO48)
- net VDD: no longer U1.2 (3V3)
- new net +3.3V: R64.1, R65.1, U1.2 (3V3)
- no-connect marks 0 -> 1
Other:
- moved on the sheet: C5, R52, U1

Commit message: Tarea 3
Parts:
- removed R1, R2: R_0603, PCM_Resistor_SMD_AKL:R_0603_1608Metric, symbol PCM_Resistor_US_AKL:R_0603
- removed USB-C_Conector: 2171820001, usb-c_footprint:MOLEX_2171820001, symbol 2171820001:2171820001
- added D18: 1N4007, Diode_SMD:D_0603_1608Metric_Pad1.05x0.95mm_HandSolder, symbol Diode:1N4007
- added D22: ESDA5V3SC5, Package_TO_SOT_SMD:SOT-23-5, symbol Power_Protection:ESDA5V3SC5
- added R1, R2, R66: R5K1, Resistor_SMD:R_0201_0603Metric, symbol Device:R_US
- added USB1: USB_C_Receptacle_USB2.0_14P, Connector_USB:USB_C_Receptacle_HRO_TYPE-C-31-M-12, symbol Connector:USB_C_Receptacle_USB2.0_14P
- C5: footprint (none) -> Capacitor_SMD:C_1206_3216Metric_Pad1.33x1.80mm_HandSolder
- R52: footprint (none) -> Resistor_SMD:R_0201_0603Metric
Connections:
- net GND: now also D22.2 (A), R1.2, R2.2, R66.2, USB1.A1 (GND), USB1.A12 (GND), USB1.B1 (GND), USB1.B12 (GND)
- net USB+: now also D22.1 (K), USB1.A6 (D+), USB1.B6 (D+)
- net USB-: now also D22.3 (K), USB1.A7 (D-), USB1.B7 (D-)
- new net: D18.2 (A), USB1.A4 (VBUS), USB1.A9 (VBUS), USB1.B4 (VBUS), USB1.B9 (VBUS)
- new net: R2.1, USB1.B5 (CC2)
- new net: R1.1, USB1.20 (SHIELD)
- new net: R66.1, USB1.A5 (CC1)
- new net USB_5V: D18.1 (K)
- new net VCC: D22.4 (K), D22.5 (K)
- no-connect marks 1 -> 10
