File: Tarea 3/Diseño PCB/PLC4UNI/input_NPN.kicad_sch (KiCad schematic)
At the start: 3 parts

Commit message: Tarea 3
Connections:
- net IN+ renamed IN
Changed lines of the file:
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@@
 		)
 	)
-	(hierarchical_label "IN+"
+	(hierarchical_label "IN"
 		(shape input)
 		(at 82.55 78.74 180)

Commit message: Tarea 3
Parts:
- added OC2, OC3: FOD817S, PCM_Package_DIP_AKL:SMDIP-4_W9.53mm, symbol PCM_Optocoupler_AKL:FOD817S
- added R5, R6, R7, R8: 2.4K, PCM_Resistor_SMD_AKL:R_0603_1608Metric, symbol PCM_Resistor_US_AKL:R_0603
Connections:
- net +3.3V: now also R6.2, R8.2
- net GND: now also OC2.3, OC3.3
- net VCC: now also R5.1, R7.1
- net IN renamed IN_NPN_A_IN
- net OUT renamed OUT_NPN_A_IN
- new net: OC3.1, R7.2
- new net: OC2.1, R5.2
- new net IN_NPN_B_IN: OC2.2
- new net IN_NPN_C_IN: OC3.2
- new net OUT_NPN_B_IN: OC2.4, R6.1
- new net OUT_NPN_C_IN: OC3.4, R8.1
Other:
- note added: "NPN INPUT_A"
- note added: "NPN INPUT_B"
- note added: "NPN INPUT_C"
- moved on the sheet: OC?, R3, R4

Commit message: Tarea 3
Parts:
- added OC12: FOD817S, PCM_Package_DIP_AKL:SMDIP-4_W9.53mm, symbol PCM_Optocoupler_AKL:FOD817S
- added R55, R56: 2.4K, PCM_Resistor_SMD_AKL:R_0603_1608Metric, symbol PCM_Resistor_US_AKL:R_0603
Connections:
- net +3.3V: now also R56.2
- net GND: now also OC12.3
- net VCC: now also R55.1
- new net: OC12.1, R55.2
- new net IN_NPN_D_IN: OC12.2
- new net OUT_NPN_D_IN: OC12.4, R56.1
Other:
- note added: "NPN INPUT_D"

Commit message: Tarea 3
Parts:
- gave numbers to parts that had none: 1
Changed lines of the file:
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@@
 		(on_board yes)
 		(dnp no)
-		(property "Reference" "OC?"
+		(property "Reference" "OC15"
 			(at 66.294 53.34 0)
 			(effects
@@
 			(project "PLC4UNI"
 				(path "/acad40d5-ac6b-4a60-8788-299f56574d0c/b188dc46-3024-4793-8d80-b9402d6c0212/16310002-096d-49db-8baf-b59f1f963118"
-					(reference "OC?")
+					(reference "OC15")
 					(unit 1)
 				)
