File: Tarea 3/Diseño PCB/PLC4UNI/output_PNP.kicad_sch (KiCad schematic)
At the start: 0 parts

Commit message: Tarea 3
Parts:
- added Q4: BC160, PCM_Package_TO_SOT_THT_AKL:TO-39-3_EBC, symbol PCM_Transistor_BJT_AKL:BC160
- added R15, R16: 2.4K, PCM_Resistor_SMD_AKL:R_0603_1608Metric, symbol PCM_Resistor_US_AKL:R_0603
Connections:
- net IN: now also R15.1
- net OUT: now also Q4.3 (C), R16.2
- new net: Q4.2 (B), R15.2
- new net GND: R16.1
- new net VCC: Q4.1 (E)

Commit message: Tarea 3
Parts:
- removed Q4: BC160, PCM_Package_TO_SOT_THT_AKL:TO-39-3_EBC, symbol PCM_Transistor_BJT_AKL:BC160
- added D5, D6, D7: LED, symbol Device:LED
- added OC10, OC11, OC9: FOD817S, PCM_Package_DIP_AKL:SMDIP-4_W9.53mm, symbol PCM_Optocoupler_AKL:FOD817S
- added Q4, Q6, Q8: PNP, symbol Simulation_SPICE:PNP
- added Q5, Q7, Q9: IRLML0040, PCM_Package_TO_SOT_SMD_AKL:SOT-23, symbol PCM_Transistor_MOSFET_AKL:IRLML0040
- added R29, R34, R38: 1.7K, PCM_Resistor_SMD_AKL:R_0603_1608Metric, symbol PCM_Resistor_US_AKL:R_0603
- added R30, R33, R37: 22K, PCM_Resistor_SMD_AKL:R_0603_1608Metric, symbol PCM_Resistor_US_AKL:R_0603
- added R31, R35: 2.4K, PCM_Resistor_SMD_AKL:R_0603_1608Metric, symbol PCM_Resistor_US_AKL:R_0603
- added R32, R36: 30K, PCM_Resistor_SMD_AKL:R_0603_1608Metric, symbol PCM_Resistor_US_AKL:R_0603
- R16: value 2.4K -> 30K
Connections:
- net OUT is gone; now on net VCC: R16.2
- net GND: now also OC10.2, OC11.2, OC9.2, Q4.3 (E), Q6.3 (E), Q8.3 (E), R30.1, R33.1, R37.1; no longer R16.1
- net VCC: now also R29.2, R32.2, R34.2, R36.2, R38.2
- net at R15.2: now also OC9.1
- net IN renamed IN_PNP_A_OUT
- new net: D5.2 (A), R29.1
- new net: OC10.1, R31.2
- new net: OC10.4, Q6.2 (B), R32.1, R33.2
- new net: OC9.4, Q4.2 (B), R16.1, R30.2
- new net: D6.2 (A), R34.1
- new net: D7.2 (A), R38.1
- new net: OC11.1, R35.2
- new net: OC11.4, Q8.2 (B), R36.1, R37.2
- new net IN_PNP_B_OUT: R31.1
- new net IN_PNP_C_OUT: R35.1
- new net OUT_PNP_A_OUT: D5.1 (K), Q4.1 (C)
- new net OUT_PNP_B_OUT: D6.1 (K), Q6.1 (C)
- new net OUT_PNP_C_OUT: D7.1 (K), Q8.1 (C)
Other:
- note added: "PNP OUTPUT_A"
- note added: "PNP OUTPUT_B"
- note added: "PNP OUTPUT_C"
- moved on the sheet: R15, R16

Commit message: Tarea 3
Parts:
- removed Q4, Q6, Q8: PNP, symbol Simulation_SPICE:PNP
Connections:
- net GND: now also OC10.3, OC11.3, OC9.3, Q5.2 (S), Q7.2 (S), Q9.2 (S)
- net OUT_PNP_A_OUT: now also Q5.3 (D)
- net OUT_PNP_B_OUT: now also Q7.3 (D)
- net OUT_PNP_C_OUT: now also Q9.3 (D)
- net at OC10.4, R32.1, R33.2: now also Q7.1 (G)
- net at OC9.4, R16.1, R30.2: now also Q5.1 (G)
- net at OC11.4, R36.1, R37.2: now also Q9.1 (G)
Other:
- moved on the sheet: Q5, Q7, Q9

Commit message: Tarea  3
Changed lines of the file:
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@@
+	)
+	(junction
+		(at 233.68 35.56)
+		(diameter 0)
+		(color 0 0 0 0)
 	)
 	(junction
@@
 	)
 	(junction
-		(at 233.68 41.91)
-		(diameter 0)
-		(color 0 0 0 0)
-	)
-	(junction
 		(at 115.57 40.64)
 		(diameter 0)
@@
 		(color 0 0 0 0)
 	)
-	(junction
-		(at 233.68 35.56)
-		(diameter 0)
-		(color 0 0 0 0)
-	)
 	(wire
 		(pts
@@
 	(wire
 		(pts
-			(xy 233.68 41.91) (xy 233.68 35.56)
-		)
-		(stroke
-			(width 0)
-			(type default)
-		)
-	)
-	(wire
-		(pts
 			(xy 115.57 40.64) (xy 115.57 46.99)
 		)
@@
 	(wire
 		(pts
-			(xy 233.68 43.18) (xy 233.68 41.91)
-		)
-		(stroke
-			(width 0)
-			(type default)
-		)
-	)
-	(wire
-		(pts
 			(xy 180.34 66.04) (xy 180.34 69.85)
 		)
@@
 	(wire
 		(pts
+			(xy 82.55 96.52) (xy 82.55 97.79)
+		)
+		(stroke
+			(width 0)
+			(type default)
+		)
+	)
+	(wire
+		(pts
+			(xy 187.96 48.26) (xy 187.96 55.88)
+		)
+		(stroke
+			(width 0)
+			(type default)
+		)
+	)
+	(wire
+		(pts
+			(xy 116.84 97.79) (xy 124.46 97.79)
+		)
+		(stroke
+			(width 0)
+			(type default)
+		)
+	)
+	(wire
+		(pts
+			(xy 116.84 104.14) (xy 116.84 97.79)
+		)
+		(stroke
+			(width 0)
+			(type default)
+		)
+	)
+	(wire
+		(pts
+			(xy 116.84 114.3) (xy 116.84 119.38)
+		)
+		(stroke
+			(width 0)
+			(type default)
+		)
+	)
+	(wire
+		(pts
+			(xy 71.12 71.12) (xy 71.12 72.39)
+		)
+		(stroke
+			(width 0)
+			(type default)
+		)
+	)
+	(wire
+		(pts
+			(xy 57.15 116.84) (xy 63.5 116.84)
+		)
+		(stroke
+			(width 0)
+			(type default)
+		)
+	)
+	(wire
+		(pts
+			(xy 199.39 58.42) (xy 199.39 66.04)
+		)
+		(stroke
+			(width 0)
+			(type default)
+		)
+	)
+	(wire
+		(pts
+			(xy 82.55 53.34) (xy 109.22 53.34)
+		)
+		(stroke
+			(width 0)
+			(type default)
+		)
+	)
+	(wire
+		(pts
+			(xy 116.84 97.79) (xy 114.3 97.79)
+		)
+		(stroke
+			(width 0)
+			(type default)
+		)
+	)
+	(wire
+		(pts
+			(xy 82.55 72.39) (xy 82.55 76.2)
+		)
+		(stroke
+			(width 0)
+			(type default)
+		)
+	)
+	(wire
+		(pts
+			(xy 82.55 53.34) (xy 82.55 55.88)
+		)
+		(stroke
+			(width 0)
+			(type default)
+		)
+	)
+	(wire
+		(pts
+			(xy 199.39 66.04) (xy 199.39 68.58)
+		)
+		(stroke
+			(width 0)
+			(type default)
+		)
+	)
+	(wire
+		(pts
+			(xy 71.12 110.49) (xy 71.12 118.11)
+		)
+		(stroke
+			(width 0)
+			(type default)
+		)
+	)
+	(wire
+		(pts
+			(xy 82.55 53.34) (xy 71.12 53.34)
+		)
+		(stroke
+			(width 0)
+			(type default)
+		)
+	)
+	(wire
+		(pts
+			(xy 199.39 48.26) (xy 187.96 48.26)
+		)
+		(stroke
+			(width 0)
+			(type default)
+		)
+	)
+	(wire
+		(pts
+			(xy 233.68 52.07) (xy 233.68 57.15)
+		)
+		(stroke
+			(width 0)
+			(type default)
+		)
+	)
+	(wire
+		(pts
+			(xy 82.55 97.79) (xy 82.55 100.33)
+		)
+		(stroke
+			(width 0)
+			(type default)
+		)
+	)
+	(wire
+		(pts
 			(xy 233.68 35.56) (xy 241.3 35.56)
 		)
@@
 	(wire
 		(pts
-			(xy 82.55 96.52) (xy 82.55 97.79)
-		)
-		(stroke
-			(width 0)
-			(type default)
-		)
-	)
-	(wire
-		(pts
-			(xy 187.96 48.26) (xy 187.96 55.88)
-		)
-		(stroke
-			(width 0)
-			(type default)
-		)
-	)
-	(wire
-		(pts
-			(xy 116.84 97.79) (xy 124.46 97.79)
-		)
-		(stroke
-			(width 0)
-			(type default)
-		)
-	)
-	(wire
-		(pts
-			(xy 116.84 104.14) (xy 116.84 97.79)
-		)
-		(stroke
-			(width 0)
-			(type default)
-		)
-	)
-	(wire
-		(pts
-			(xy 116.84 114.3) (xy 116.84 119.38)
-		)
-		(stroke
-			(width 0)
-			(type default)
-		)
-	)
-	(wire
-		(pts
-			(xy 71.12 71.12) (xy 71.12 72.39)
-		)
-		(stroke
-			(width 0)
-			(type default)
-		)
-	)
-	(wire
-		(pts
-			(xy 57.15 116.84) (xy 63.5 116.84)
-		)
-		(stroke
-			(width 0)
-			(type default)
-		)
-	)
-	(wire
-		(pts
-			(xy 199.39 58.42) (xy 199.39 66.04)
-		)
-		(stroke
-			(width 0)
-			(type default)
-		)
-	)
-	(wire
-		(pts
-			(xy 82.55 53.34) (xy 109.22 53.34)
-		)
-		(stroke
-			(width 0)
-			(type default)
-		)
-	)
-	(wire
-		(pts
-			(xy 116.84 97.79) (xy 114.3 97.79)
-		)
-		(stroke
-			(width 0)
-			(type default)
-		)
-	)
-	(wire
-		(pts
-			(xy 82.55 72.39) (xy 82.55 76.2)
-		)
-		(stroke
-			(width 0)
-			(type default)
-		)
-	)
-	(wire
-		(pts
-			(xy 82.55 53.34) (xy 82.55 55.88)
-		)
-		(stroke
-			(width 0)
-			(type default)
-		)
-	)
-	(wire
-		(pts
-			(xy 199.39 66.04) (xy 199.39 68.58)
-		)
-		(stroke
-			(width 0)
-			(type default)
-		)
-	)
-	(wire
-		(pts
-			(xy 71.12 110.49) (xy 71.12 118.11)
-		)
-		(stroke
-			(width 0)
-			(type default)
-		)
-	)
-	(wire
-		(pts
-			(xy 82.55 53.34) (xy 71.12 53.34)
-		)
-		(stroke
-			(width 0)
-			(type default)
-		)
-	)
-	(wire
-		(pts
-			(xy 199.39 48.26) (xy 187.96 48.26)
-		)
-		(stroke
-			(width 0)
-			(type default)
-		)
-	)
-	(wire
-		(pts
-			(xy 233.68 52.07) (xy 233.68 57.15)
-		)
-		(stroke
-			(width 0)
-			(type default)
-		)
-	)
-	(wire
-		(pts
-			(xy 82.55 97.79) (xy 82.55 100.33)
-		)
-		(stroke
-			(width 0)
-			(type default)
-		)
-	)
-	(wire
-		(pts
 			(xy 82.55 97.79) (xy 91.44 97.79)
 		)
@@
 	(wire
 		(pts
+			(xy 233.68 35.56) (xy 233.68 41.91)
+		)
+		(stroke
+			(width 0)
+			(type default)
+		)
+	)
+	(wire
+		(pts
 			(xy 82.55 110.49) (xy 82.55 113.03)
 		)
@@
 	(wire
 		(pts
-			(xy 233.68 35.56) (xy 231.14 35.56)
-		)
-		(stroke
+			(xy 231.14 35.56) (xy 233.68 35.56)
+		)
+		(stroke

Commit message: Tarea 3
Parts:
- D5, D6, D7: footprint (none) -> LED_SMD:LED_0603_1608Metric
Changed lines of the file:
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@@
 			)
 		)
-		(property "Footprint" ""
+		(property "Footprint" "LED_SMD:LED_0603_1608Metric"
 			(at 110.49 40.64 0)
 			(effects
@@
 			)
 		)
-		(property "Footprint" ""
+		(property "Footprint" "LED_SMD:LED_0603_1608Metric"
 			(at 110.49 97.79 0)
 			(effects
@@
 			)
 		)
-		(property "Footprint" ""
+		(property "Footprint" "LED_SMD:LED_0603_1608Metric"
 			(at 227.33 35.56 0)
 			(effects
