File: Tarea 3/Diseño PCB/PLC4UNI/Board-PLC4UNI-G1w.kicad_sch (KiCad schematic)
At the start: 0 parts

Commit message: Tarea 3
Other:
- added sheet input_PNP1 (input_PNP.kicad_sch)
- added sheet input_PNP2 (input_PNP.kicad_sch)
- sheet input_NPN ports: added IN; removed IN+
- sheet input_NPN1 ports: added IN; removed IN+
- sheet input_NPN2 ports: added IN; removed IN+
Changed lines of the file:
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@@
 			)
 		)
-		(pin "IN+" input
+		(pin "OUT" output
+			(at 31.75 19.05 0)
+			(effects
+				(font
+					(size 1.27 1.27)
+				)
+				(justify right)
+			)
+		)
+		(pin "IN" input
 			(at 15.24 19.05 180)
 			(effects
@@
 				)
 				(justify left)
-			)
-		)
-		(pin "OUT" output
-			(at 31.75 19.05 0)
-			(effects
-				(font
-					(size 1.27 1.27)
-				)
-				(justify right)
 			)
 		)
@@
 			)
 		)
-		(pin "IN+" input
+		(pin "OUT" output
+			(at 31.75 29.21 0)
+			(effects
+				(font
+					(size 1.27 1.27)
+				)
+				(justify right)
+			)
+		)
+		(pin "IN" input
 			(at 15.24 29.21 180)
 			(effects
@@
 				)
 				(justify left)
-			)
-		)
-		(pin "OUT" output
-			(at 31.75 29.21 0)
-			(effects
-				(font
-					(size 1.27 1.27)
-				)
-				(justify right)
 			)
 		)
@@
 	)
 	(sheet
+		(at 74.93 26.67)
+		(size 16.51 5.08)
+		(exclude_from_sim no)
+		(in_bom yes)
+		(on_board yes)
+		(dnp no)
+		(fields_autoplaced yes)
+		(stroke
+			(width 0.1524)
+			(type solid)
+		)
+		(fill
+			(color 0 0 0 0.0000)
+		)
+		(property "Sheetname" "input_PNP1"
+			(at 74.93 25.9584 0)
+			(effects
+				(font
+					(size 1.27 1.27)
+				)
+				(justify left bottom)
+			)
+		)
+		(property "Sheetfile" "input_PNP.kicad_sch"
+			(at 74.93 32.3346 0)
+			(effects
+				(font
+					(size 1.27 1.27)
+				)
+				(justify left top)
+			)
+		)
+		(pin "IN" input
+			(at 74.93 29.21 180)
+			(effects
+				(font
+					(size 1.27 1.27)
+				)
+				(justify left)
+			)
+		)
+		(pin "OUT" output
+			(at 91.44 29.21 0)
+			(effects
+				(font
+					(size 1.27 1.27)
+				)
+				(justify right)
+			)
+		)
+		(instances
+			(project "PLC4UNI"
+				(path "/acad40d5-ac6b-4a60-8788-299f56574d0c/b188dc46-3024-4793-8d80-b9402d6c0212"
+					(page "15")
+				)
+			)
+		)
+	)
+	(sheet
 		(at 104.14 16.51)
 		(size 16.51 5.08)
@@
 	)
 	(sheet
+		(at 74.93 38.1)
+		(size 16.51 5.08)
+		(exclude_from_sim no)
+		(in_bom yes)
+		(on_board yes)
+		(dnp no)
+		(fields_autoplaced yes)
+		(stroke
+			(width 0.1524)
+			(type solid)
+		)
+		(fill
+			(color 0 0 0 0.0000)
+		)
+		(property "Sheetname" "input_PNP2"
+			(at 74.93 37.3884 0)
+			(effects
+				(font
+					(size 1.27 1.27)
+				)
+				(justify left bottom)
+			)
+		)
+		(property "Sheetfile" "input_PNP.kicad_sch"
+			(at 74.93 43.7646 0)
+			(effects
+				(font
+					(size 1.27 1.27)
+				)
+				(justify left top)
+			)
+		)
+		(pin "IN" input
+			(at 74.93 40.64 180)
+			(effects
+				(font
+					(size 1.27 1.27)
+				)
+				(justify left)
+			)
+		)
+		(pin "OUT" output
+			(at 91.44 40.64 0)
+			(effects
+				(font
+					(size 1.27 1.27)
+				)
+				(justify right)
+			)
+		)
+		(instances
+			(project "PLC4UNI"
+				(path "/acad40d5-ac6b-4a60-8788-299f56574d0c/b188dc46-3024-4793-8d80-b9402d6c0212"
+					(page "16")
+				)
+			)
+		)
+	)
+	(sheet
 		(at 74.93 16.51)
 		(size 16.51 5.08)
@@
 			)
 		)
-		(pin "IN+" input
+		(pin "OUT" output
+			(at 31.75 39.37 0)
+			(effects
+				(font
+					(size 1.27 1.27)
+				)
+				(justify right)
+			)
+		)
+		(pin "IN" input
 			(at 15.24 39.37 180)
 			(effects
@@
 			)
 		)
-		(pin "OUT" output
-			(at 31.75 39.37 0)
-			(effects
-				(font
-					(size 1.27 1.27)
-				)
-				(justify right)
-			)
-		)

Commit message: Tarea 3
Other:
- removed sheet input_NPN1
- removed sheet input_NPN2
- removed sheet input_PNP1
- removed sheet input_PNP2
- sheet input_NPN ports: added IN_NPN_A_IN, IN_NPN_B_IN, IN_NPN_C_IN, OUT_NPN_A_IN, OUT_NPN_B_IN, OUT_NPN_C_IN; removed IN, OUT
- sheet input_PNP ports: added IN_PNP_A_IN, IN_PNP_B_IN, IN_PNP_C_IN, OUT_PNP_A_IN, OUT_PNP_B_IN, OUT_PNP_C_IN; removed IN, OUT
- sheet output_NPN ports: added IN_NPN_A_OUT, IN_NPN_B_OUT, IN_NPN_C_OUT, OUT_NPN_A_OUT, OUT_NPN_B_OUT, OUT_NPN_C_OUT; removed IN, OUT
- sheet output_PNP ports: added IN_PNP_A_OUT, IN_PNP_B_OUT, IN_PNP_C_OUT, OUT_PNP_A_OUT, OUT_PNP_B_OUT, OUT_PNP_C_OUT; removed IN, OUT

Commit message: Tarea 3
Other:
- removed sheet rs485_module_protect
- added sheet 0-10V_Output (0-10V_Output.kicad_sch)
- added sheet 4-20mA (4-20mA.kicad_sch)
- added sheet PowerSupply (PowerSupply.kicad_sch)
- added sheet RS485 (RS485.kicad_sch)
- sheet PLC4UNI_CPU ports: added ESP32_UART_A, ESP32_UART_B, FROMESP_OUT_IN-NPN_A, FROMESP_OUT_IN-NPN_B, FROMESP_OUT_IN-NPN_C, FROMESP_OUT_IN-PNP_A, FROMESP_OUT_IN-PNP_B, FROMESP_OUT_IN-PNP_C, FROMESP_SCLK_C, FROMESP_SCLK_V, FROMESP_SDA_C, FROMESP_SDA_V, FROMESP_SEL_VOUT; removed micro_RS485_control, micro_RS485_rx, micro_RS485_tx

Commit message: Tarea 3
Other:
- sheet PLC4UNI_CPU ports: added FROMESP_IN_OUT-NPN_A, FROMESP_IN_OUT-NPN_B, FROMESP_IN_OUT-NPN_C, FROMESP_IN_OUT-PNP_A, FROMESP_IN_OUT-PNP_B, FROMESP_IN_OUT-PNP_C; removed none

Commit message: Tarea 3
Other:
- added sheet OUT_RLY_A (OUT_RLY_A.kicad_sch)
- added sheet OUT_RLY_B (OUT_RLY_B.kicad_sch)
- sheet PLC4UNI_CPU ports: added RLY_A_INR, RLY_B_INR; removed none

Commit message: Tarea 3
Other:
- sheet 4-20mA renamed 4-20mA_Output
- added sheet 0-10_Input (0-10_Input.kicad_sch)
- added sheet 4-20mA_Input (4-20mA_Input.kicad_sch)
- sheet 0-10V_Output ports: added SEL, VOLTAGE_AOUTPUT; removed 0-10V_OUT_1, ESP32_SEL_VOUT
- sheet 4-20mA_Output: file 4-20mA.kicad_sch -> 4-20mA_Output.kicad_sch
- sheet PLC4UNI_CPU ports: added FROMESP_IN_OUT-NPN_D, FROMESP_OUT_IN-NPN_D, FROMESP_OUT_IN-PNP_D, FROMESP_SCLK, FROMESP_SDA, FROMESP_Voltage_Input; removed FROMESP_SCLK_C, FROMESP_SCLK_V, FROMESP_SDA_C, FROMESP_SDA_V
- sheet input_NPN ports: added IN_NPN_D_IN, OUT_NPN_D_IN; removed none
- sheet input_PNP ports: added IN_PNP_D_IN, OUT_PNP_D_IN; removed none
- sheet output_NPN ports: added IN_NPN_D_OUT, OUT_NPN_D_OUT; removed none

Commit message: Tarea  3
Other:
- sheet PLC4UNI_CPU ports: added FROMESP_4-20mA_Input; removed none
Changed lines of the file:
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@@
+	(wire
+		(pts
+			(xy 194.31 92.71) (xy 198.12 92.71)
+		)
+		(stroke
+			(width 0)
+			(type default)
+		)
+	)
 	(wire
 		(pts
@@
 	(wire
 		(pts
+			(xy 198.12 104.14) (xy 201.93 104.14)
+		)
+		(stroke
+			(width 0)
+			(type default)
+		)
+	)
+	(wire
+		(pts
 			(xy 118.11 35.56) (xy 120.65 35.56)
 		)
@@
 		(pts
 			(xy 115.57 77.47) (xy 139.7 77.47)
+		)
+		(stroke
+			(width 0)
+			(type default)
+		)
+	)
+	(wire
+		(pts
+			(xy 198.12 92.71) (xy 198.12 104.14)
 		)
 		(stroke
@@
 			(effects
 				(font
+					(size 1.27 1.27)
+				)
+				(justify right)
+			)
+		)
+		(pin "FROMESP_4-20mA_Input" input
+			(at 194.31 92.71 0)
+			(effects
+				(font

Commit message: tarea 3 - update
Changed lines of the file:
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@@
 			)
 		)
-		(pin "UART_IN" input
+		(pin "UART_IN" bidirectional
 			(at 201.93 50.8 180)
 			(effects
@@
 			)
 		)
-		(pin "UART_OUT" output
+		(pin "UART_OUT" bidirectional
 			(at 201.93 53.34 180)
 			(effects
