File: Tarea 3/Diseño PCB/PLC4UNI/PLC4UNI.kicad_pcb (KiCad board)
At the start: 2 copper layers, 2 parts, among them J2 Screw_Terminal_01x18

Commit message: Tarea  3
Parts:
- moved J2 1.55 mm to (71.0, 111.5)
- moved J2 1.00 mm to (71.0, 39.5)
Other:
- copper layers 2 -> 4
Changed lines of the file:
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@@
 	(layers
 		(0 "F.Cu" signal)
+		(4 "In1.Cu" signal)
+		(6 "In2.Cu" signal)
 		(2 "B.Cu" signal)
 		(9 "F.Adhes" user "F.Adhesive")
@@
 	)
 	(setup
+		(stackup
+			(layer "F.SilkS"
+				(type "Top Silk Screen")
+			)
+			(layer "F.Paste"
+				(type "Top Solder Paste")
+			)
+			(layer "F.Mask"
+				(type "Top Solder Mask")
+				(thickness 0.01)
+			)
+			(layer "F.Cu"
+				(type "copper")
+				(thickness 0.035)
+			)
+			(layer "dielectric 1"
+				(type "prepreg")
+				(thickness 0.1)
+				(material "FR4")
+				(epsilon_r 4.5)
+				(loss_tangent 0.02)
+			)
+			(layer "In1.Cu"
+				(type "copper")
+				(thickness 0.035)
+			)
+			(layer "dielectric 2"
+				(type "core")
+				(thickness 1.24)
+				(material "FR4")
+				(epsilon_r 4.5)
+				(loss_tangent 0.02)
+			)
+			(layer "In2.Cu"
+				(type "copper")
+				(thickness 0.035)
+			)
+			(layer "dielectric 3"
+				(type "prepreg")
+				(thickness 0.1)
+				(material "FR4")
+				(epsilon_r 4.5)
+				(loss_tangent 0.02)
+			)
+			(layer "B.Cu"
+				(type "copper")
+				(thickness 0.035)
+			)
+			(layer "B.Mask"
+				(type "Bottom Solder Mask")
+				(thickness 0.01)
+			)
+			(layer "B.Paste"
+				(type "Bottom Solder Paste")
+			)
+			(layer "B.SilkS"
+				(type "Bottom Silk Screen")
+			)
+			(copper_finish "None")
+			(dielectric_constraints no)
+		)
 		(pad_to_mask_clearance 0)
 		(allow_soldermask_bridges_in_footprints no)
 		(tenting front back)
+		(grid_origin 63 115.5)
 		(pcbplotparams
 			(layerselection 0x00000000_00000000_55555555_5755f5ff)
@@
 	(footprint "TerminalBlock:TerminalBlock_MaiXu_MX126-5.0-18P_1x18_P5.00mm"
 		(layer "F.Cu")
-		(at 70.5 112.9675)
+		(at 71 111.5)
 		(descr "terminal block MaiXu MX126-5.0-18P, 18 pins, pitch 5mm, size 90.5x7.8mm, drill diameter 1.3mm, pad diameter 2.8mm, https://www.lcsc.com/datasheet/lcsc_datasheet_2309150913_MAX-MX126-5-0-03P-GN01-Cu-S-A_C5188435.pdf, script-generated using https://gitlab.com/kicad/libraries/kicad-footprint-generator/-/tree/master/scripts/TerminalBlock_MaiXu")
 		(tags "THT terminal block MaiXu MX126-5.0-18P pitch 5mm size 90.5x7.8mm drill 1.3mm pad 2.8mm")
@@
 	(footprint "TerminalBlock:TerminalBlock_MaiXu_MX126-5.0-18P_1x18_P5.00mm"
 		(layer "F.Cu")
-		(at 70 39.5)
+		(at 71 39.5)
 		(descr "terminal block MaiXu MX126-5.0-18P, 18 pins, pitch 5mm, size 90.5x7.8mm, drill diameter 1.3mm, pad diameter 2.8mm, https://www.lcsc.com/datasheet/lcsc_datasheet_2309150913_MAX-MX126-5-0-03P-GN01-Cu-S-A_C5188435.pdf, script-generated using https://gitlab.com/kicad/libraries/kicad-footprint-generator/-/tree/master/scripts/TerminalBlock_MaiXu")
 		(tags "THT terminal block MaiXu MX126-5.0-18P pitch 5mm size 90.5x7.8mm drill 1.3mm pad 2.8mm")
@@
 	)
 	(gr_line
-		(start 62.895476 81.1)
-		(end 62.895476 115.682919)
+		(start 63 80.917081)
+		(end 63 115.5)
 		(stroke
 			(width 0.2)
@@
 	)
 	(gr_line
-		(start 62.895476 115.682919)
-		(end 162.822014 115.682919)
+		(start 63 115.5)
+		(end 162.926538 115.5)
 		(stroke
 			(width 0.2)

Commit message: Tarea 3
Parts:
- removed the J2 at (71.0, 111.5)
- removed the J2 at (71.0, 39.5)
- added C1: 100pF, PCM_Capacitor_SMD_AKL:C_0603_1608Metric, F.Cu at (-45.1, 150.7)
- added C10: 100nF, PCM_Capacitor_SMD_AKL:C_0603_1608Metric, F.Cu at (-25.0, 57.4)
- added C12: 100nF, PCM_Capacitor_SMD_AKL:C_0603_1608Metric, F.Cu at (-29.9, 92.2)
- added C13: 220pF, PCM_Capacitor_SMD_AKL:C_0603_1608Metric, F.Cu at (-37.1, 125.7)
- added C14: 1uF, PCM_Capacitor_SMD_AKL:C_0603_1608Metric, F.Cu at (-37.1, 128.4)
- added C15: 0.1uF, PCM_Capacitor_SMD_AKL:C_0603_1608Metric, F.Cu at (-37.1, 131.2)
- added C2: 22uF, PCM_4ms_Capacitor:C_0805, F.Cu at (-49.4, 150.8)
- added C3: 10uF, PCM_Capacitor_SMD_AKL:C_1206_3216Metric, F.Cu at (-39.9, 155.7)
- added C4: 100nF, PCM_Capacitor_SMD_AKL:C_0603_1608Metric, F.Cu at (-45.1, 153.4)
- added C5: C, Capacitor_SMD:C_1206_3216Metric_Pad1.33x1.80mm_HandSolder, F.Cu at (-112.9, 116.7)
- added C6: 22uF, PCM_4ms_Capacitor:C_0805, F.Cu at (-49.4, 153.6)
- added C7: 10uF, PCM_Capacitor_SMD_AKL:C_0603_1608Metric, F.Cu at (-24.3, 155.5)
- added C8: 100nF, Capacitor_SMD:C_0805_2012Metric, F.Cu at (-32.4, 84.3)
- added C9: 1uF, Capacitor_SMD:C_0805_2012Metric_Pad1.18x1.45mm_HandSolder, F.Cu at (-32.2, 81.2)
- added D1: SMBJ12CA, PCM_Diode_SMD_AKL:D_SMB_TVS, F.Cu at (-30.5, 146.6)
- added D10: 1N4001, Diode_THT:D_DO-41_SOD81_P10.16mm_Horizontal, F.Cu at (-38.0, 116.1)
- added D11: SMF24A, Diode_SMD:D_SMF, F.Cu at (-37.5, 81.4)
- added D12: LED, LED_SMD:LED_0603_1608Metric, F.Cu at (-107.1, 147.5)
- added D13: SMAJ5.0A, PCM_Diode_SMD_AKL:D_SMA, F.Cu at (-36.3, 90.5)
- added D14: SMAJ5.0A, PCM_Diode_SMD_AKL:D_SMA, F.Cu at (-31.3, 53.3)
- added D15: SMAJ5.0A, PCM_Diode_SMD_AKL:D_SMA, F.Cu at (-31.3, 58.8)
- added D16: SMAJ5.0A, PCM_Diode_SMD_AKL:D_SMA, F.Cu at (-30.6, 152.2)
- added D17: BZT52C12_C2891780, Diode_SMD:D_SOD-123, F.Cu at (-36.0, 136.9)
- added D18: 1N4007, Diode_SMD:D_0603_1608Metric_Pad1.05x0.95mm_HandSolder, F.Cu at (-103.6, 116.3)
- added D19: SMAJ5.0A, PCM_Diode_SMD_AKL:D_SMA, F.Cu at (-36.3, 96.0)
- added D2: LED, LED_SMD:LED_0603_1608Metric, F.Cu at (-107.1, 139.7)
- added D20: SMAJ33A, Diode_SMD:D_SMA, F.Cu at (-47.4, 126.6)
- added D21: MRA4007T3G, Diode_SMD:D_SMA, F.Cu at (-47.4, 131.2)
- added D22: ESDA5V3SC5, Package_TO_SOT_SMD:SOT-23-5, F.Cu at (-113.3, 120.8)
- added D3: LED, LED_SMD:LED_0603_1608Metric, F.Cu at (-107.1, 142.3)
- added D4: LED, LED_SMD:LED_0603_1608Metric, F.Cu at (-107.1, 144.9)
- added D5: LED, LED_SMD:LED_0603_1608Metric, F.Cu at (-59.0, 102.7)
- added D6: LED, LED_SMD:LED_0603_1608Metric, F.Cu at (-59.0, 105.3)
- added D7: LED, LED_SMD:LED_0603_1608Metric, F.Cu at (-59.0, 107.9)
- added D8: SM712, PCM_Package_TO_SOT_SMD_AKL:SOT-23, F.Cu at (-24.1, 151.8)
- added D9: 1N4001, Diode_THT:D_DO-41_SOD81_P10.16mm_Horizontal, F.Cu at (-65.5, 143.1)
- added J1: Screw_Terminal_01x18, TerminalBlock:TerminalBlock_MaiXu_MX126-5.0-18P_1x18_P5.00mm, F.Cu at (71.0, 40.0)
- added J2: Screw_Terminal_01x18, TerminalBlock:TerminalBlock_MaiXu_MX126-5.0-18P_1x18_P5.00mm, F.Cu at (71.0, 110.5)
- added K1: G5Q-1, Relay_THT:Relay_SPDT_Omron-G5Q-1, F.Cu at (-49.0, 111.5)
- added K2: G5Q-1, Relay_THT:Relay_SPDT_Omron-G5Q-1, F.Cu at (-76.5, 138.5)
- added L1: 6.8uH, Inductor_SMD:L_Chilisin_BMRA00040420, F.Cu at (-48.1, 146.5)
- added OC1: FOD817S, PCM_Package_DIP_AKL:SMDIP-4_W9.53mm, F.Cu at (-115.7, 130.8)
- added OC10: FOD817S, PCM_Package_DIP_AKL:SMDIP-4_W9.53mm, F.Cu at (-72.4, 111.4)
- added OC11: FOD817S, PCM_Package_DIP_AKL:SMDIP-4_W9.53mm, F.Cu at (-72.4, 118.0)
- added OC12: FOD817S, PCM_Package_DIP_AKL:SMDIP-4_W9.53mm, F.Cu at (-72.4, 89.4)
- added OC13: FOD817S, PCM_Package_DIP_AKL:SMDIP-4_W9.53mm, F.Cu at (-53.1, 96.1)
- added OC14: FOD817S, PCM_Package_DIP_AKL:SMDIP-4_W9.53mm, F.Cu at (-115.7, 150.8)
- added OC15: FOD817S, PCM_Package_DIP_AKL:SMDIP-4_W9.53mm, F.Cu at (-72.4, 96.1)
- added OC2: FOD817S, PCM_Package_DIP_AKL:SMDIP-4_W9.53mm, F.Cu at (-72.4, 76.1)
- added OC3: FOD817S, PCM_Package_DIP_AKL:SMDIP-4_W9.53mm, F.Cu at (-72.4, 82.8)
- added OC4: FOD817S, PCM_Package_DIP_AKL:SMDIP-4_W9.53mm, F.Cu at (-53.1, 76.1)
- added OC5: FOD817S, PCM_Package_DIP_AKL:SMDIP-4_W9.53mm, F.Cu at (-53.1, 82.8)
- added OC6: FOD817S, PCM_Package_DIP_AKL:SMDIP-4_W9.53mm, F.Cu at (-53.1, 89.4)
- added OC7: FOD817S, PCM_Package_DIP_AKL:SMDIP-4_W9.53mm, F.Cu at (-115.7, 137.5)
- added OC8: FOD817S, PCM_Package_DIP_AKL:SMDIP-4_W9.53mm, F.Cu at (-115.7, 144.1)
- added OC9: FOD817S, PCM_Package_DIP_AKL:SMDIP-4_W9.53mm, F.Cu at (-72.4, 104.7)
- added Q1: BC108A, PCM_Package_TO_SOT_THT_AKL:TO-18-3_EBC, F.Cu at (-127.2, 131.6)
- added Q10: IRLML6402TRPBF-JSM, PCM_4ms_Package_SOT:SOT-23, F.Cu at (-41.1, 137.5)
- added Q2: BC108A, PCM_Package_TO_SOT_THT_AKL:TO-18-3_EBC, F.Cu at (-127.2, 139.3)
- added Q3: BC108A, PCM_Package_TO_SOT_THT_AKL:TO-18-3_EBC, F.Cu at (-127.2, 147.0)
- added Q4: TIP41, Package_TO_SOT_THT:TO-220-3_Vertical, F.Cu at (-75.7, 144.9)
- added Q5: IRLML0040, PCM_Package_TO_SOT_SMD_AKL:SOT-23, F.Cu at (-63.5, 103.7)
- added Q6: TIP41, Package_TO_SOT_THT:TO-220-3_Vertical, F.Cu at (-48.2, 117.9)
- added Q7: IRLML0040, PCM_Package_TO_SOT_SMD_AKL:SOT-23, F.Cu at (-63.5, 108.5)
- added Q8: BC108A, PCM_Package_TO_SOT_THT_AKL:TO-18-3_EBC, F.Cu at (-127.2, 154.7)
- added Q9: IRLML0040, PCM_Package_TO_SOT_SMD_AKL:SOT-23, F.Cu at (-63.5, 113.2)
- added R1: R5K1, Resistor_SMD:R_0201_0603Metric, F.Cu at (-117.1, 115.9)
- added R10: 100, PCM_Resistor_SMD_AKL:R_0603_1608Metric, F.Cu at (-107.1, 131.6)
- added R11: 2.4K, PCM_Resistor_SMD_AKL:R_0603_1608Metric, F.Cu at (-44.5, 74.1)
- added R12: 2.4K, PCM_Resistor_SMD_AKL:R_0603_1608Metric, F.Cu at (-44.5, 76.9)
- added R13: 2.4K, PCM_Resistor_SMD_AKL:R_0603_1608Metric, F.Cu at (-44.5, 79.6)
- added R14: 2.4K, PCM_Resistor_SMD_AKL:R_0603_1608Metric, F.Cu at (-44.5, 82.3)
- added R15: 2.4K, PCM_Resistor_SMD_AKL:R_0603_1608Metric, F.Cu at (-63.8, 116.9)
- added R16: 30K, PCM_Resistor_SMD_AKL:R_0603_1608Metric, F.Cu at (-63.8, 119.6)
- added R17: 100K, PCM_Resistor_SMD_AKL:R_0603_1608Metric, F.Cu at (-107.1, 134.3)
- added R18: 100, PCM_Resistor_SMD_AKL:R_0603_1608Metric, F.Cu at (-107.1, 137.0)
- added R19: 2.4K, PCM_Resistor_SMD_AKL:R_0603_1608Metric, F.Cu at (-103.0, 128.9)
- added R2: R5K1, Resistor_SMD:R_0201_0603Metric, F.Cu at (-117.1, 117.7)
- added R20: 100K, PCM_Resistor_SMD_AKL:R_0603_1608Metric, F.Cu at (-103.0, 131.6)
- added R21: 2.4K, PCM_Resistor_SMD_AKL:R_0603_1608Metric, F.Cu at (-44.5, 85.0)
- added R22: 2.4K, PCM_Resistor_SMD_AKL:R_0603_1608Metric, F.Cu at (-44.5, 87.7)
- added R23: 100, PCM_Resistor_SMD_AKL:R_0603_1608Metric, F.Cu at (-103.0, 134.3)
- added R24: 100, PCM_Resistor_SMD_AKL:R_0603_1608Metric, F.Cu at (-103.0, 137.0)
- added R25: 2.4K, PCM_Resistor_SMD_AKL:R_0603_1608Metric, F.Cu at (-98.9, 128.9)
- added R26: 100K, PCM_Resistor_SMD_AKL:R_0603_1608Metric, F.Cu at (-98.9, 131.6)
- added R27: 100, PCM_Resistor_SMD_AKL:R_0603_1608Metric, F.Cu at (-98.9, 134.3)
- added R28: 100, PCM_Resistor_SMD_AKL:R_0603_1608Metric, F.Cu at (-98.9, 137.0)
- added R29: 1.7K, PCM_Resistor_SMD_AKL:R_0603_1608Metric, F.Cu at (-63.8, 122.3)
- added R3: 2.4K, PCM_Resistor_SMD_AKL:R_0603_1608Metric, F.Cu at (-63.8, 74.1)
- added R30: 22K, PCM_Resistor_SMD_AKL:R_0603_1608Metric, F.Cu at (-63.8, 125.1)
- added R31: 2.4K, PCM_Resistor_SMD_AKL:R_0603_1608Metric, F.Cu at (-59.6, 116.9)
- added R32: 30K, PCM_Resistor_SMD_AKL:R_0603_1608Metric, F.Cu at (-59.6, 119.6)
- added R33: 22K, PCM_Resistor_SMD_AKL:R_0603_1608Metric, F.Cu at (-59.6, 122.3)
- added R34: 1.7K, PCM_Resistor_SMD_AKL:R_0603_1608Metric, F.Cu at (-59.6, 125.1)
- added R35: 2.4K, PCM_Resistor_SMD_AKL:R_0603_1608Metric, F.Cu at (-55.5, 116.9)
- added R36: 30K, PCM_Resistor_SMD_AKL:R_0603_1608Metric, F.Cu at (-55.5, 119.6)
- added R37: 22K, PCM_Resistor_SMD_AKL:R_0603_1608Metric, F.Cu at (-55.5, 122.3)
- added R38: 1.7K, PCM_Resistor_SMD_AKL:R_0603_1608Metric, F.Cu at (-55.5, 125.1)
- added R39: 47K, PCM_Resistor_SMD_AKL:R_0603_1608Metric, F.Cu at (-24.2, 145.1)
- added R4: 2.4K, PCM_Resistor_SMD_AKL:R_0603_1608Metric, F.Cu at (-63.8, 76.9)
- added R40: 47K, PCM_Resistor_SMD_AKL:R_0603_1608Metric, F.Cu at (-24.2, 147.8)
- added R41: 196K, PCM_Resistor_SMD_AKL:R_0603_1608Metric, F.Cu at (-42.6, 145.1)
- added R42: 62K, PCM_Resistor_SMD_AKL:R_0603_1608Metric, F.Cu at (-42.6, 147.8)
- added R43: 4.7K, PCM_Resistor_SMD_AKL:R_0603_1608Metric, F.Cu at (-41.3, 125.7)
- added R44: 10k, Resistor_SMD:R_0603_1608Metric, F.Cu at (-38.4, 84.3)
- added R45: 2.4K, PCM_Resistor_SMD_AKL:R_0603_1608Metric, F.Cu at (-94.7, 128.9)
- added R46: 4.7K, PCM_Resistor_SMD_AKL:R_0603_1608Metric, F.Cu at (-41.3, 128.4)
- added R47: 100K, PCM_Resistor_SMD_AKL:R_0603_1608Metric, F.Cu at (-41.3, 131.1)
- added R48: 100K, PCM_Resistor_SMD_AKL:R_0603_1608Metric, F.Cu at (-94.7, 131.6)
- added R49: 15, PCM_Resistor_SMD_AKL:R_0805_2012Metric, F.Cu at (-36.7, 140.1)
- added R5: 2.4K, PCM_Resistor_SMD_AKL:R_0603_1608Metric, F.Cu at (-63.8, 79.6)
- added R50: 100, PCM_Resistor_SMD_AKL:R_0603_1608Metric, F.Cu at (-94.7, 134.3)
- added R51: 2.5K, PCM_Resistor_SMD_AKL:R_0603_1608Metric, F.Cu at (-41.3, 133.9)
- added R52: R_US, Resistor_SMD:R_0201_0603Metric, F.Cu at (-117.1, 119.4)
- added R53: R_US, Resistor_SMD:R_0201_0603Metric, F.Cu at (-56.6, 146.1)
- added R54: R_US, Resistor_SMD:R_0201_0603Metric, F.Cu at (-29.1, 119.1)
- added R55: 2.4K, PCM_Resistor_SMD_AKL:R_0603_1608Metric, F.Cu at (-63.8, 90.5)
- added R56: 2.4K, PCM_Resistor_SMD_AKL:R_0603_1608Metric, F.Cu at (-63.8, 93.2)
- added R57: 2.4K, PCM_Resistor_SMD_AKL:R_0603_1608Metric, F.Cu at (-44.5, 90.5)
- added R58: 2.4K, Resistor_SMD:R_0201_0603Metric, F.Cu at (-45.3, 92.7)
- added R59: 100, PCM_Resistor_SMD_AKL:R_0603_1608Metric, F.Cu at (-94.7, 137.0)
- added R6: 2.4K, PCM_Resistor_SMD_AKL:R_0603_1608Metric, F.Cu at (-63.8, 82.3)
- added R60: 25K, PCM_Resistor_SMD_AKL:R_0603_1608Metric, F.Cu at (-25.1, 51.9)
- added R61: 10K, PCM_Resistor_SMD_AKL:R_0603_1608Metric, F.Cu at (-25.1, 54.6)
- added R62: 145, PCM_Resistor_SMD_AKL:R_0805_2012Metric, F.Cu at (-29.8, 89.3)
- added R63: 1k, PCM_Resistor_SMD_AKL:R_0603_1608Metric, F.Cu at (-30.0, 95.0)
- added R64: 4.7k, Resistor_SMD:R_0603_1608Metric, F.Cu at (-107.9, 116.3)
- added R65: 4.7k, Resistor_SMD:R_0603_1608Metric, F.Cu at (-107.9, 118.8)
- added R66: R5K1, Resistor_SMD:R_0201_0603Metric, F.Cu at (-117.1, 121.2)
- added R7: 2.4K, PCM_Resistor_SMD_AKL:R_0603_1608Metric, F.Cu at (-63.8, 85.0)
- added R8: 2.4K, PCM_Resistor_SMD_AKL:R_0603_1608Metric, F.Cu at (-63.8, 87.7)
- added R9: 2.4K, PCM_Resistor_SMD_AKL:R_0603_1608Metric, F.Cu at (-107.1, 128.9)
- added U1: ESP32-S3-WROOM-1, RF_Module:ESP32-S3-WROOM-1, F.Cu at (-105.5, 101.1)
- added U18: TLP290, Package_SO:SOP-4_4.4x2.6mm_P1.27mm, F.Cu at (-62.6, 147.3)
- added U19: ~, Package_SO:SOIC-8_5.3x5.3mm_P1.27mm, F.Cu at (-35.2, 76.3)
- added U2: AP63203WU, Package_TO_SOT_SMD:TSOT-23-6, F.Cu at (-40.4, 151.7)
- added U3: GP8303-TC50-EW, Package_SO:SSOP-10_3.9x4.9mm_P1.00mm, F.Cu at (-47.6, 136.9)
- added U4: TLP290, Package_SO:SOP-4_4.4x2.6mm_P1.27mm, F.Cu at (-35.1, 120.3)
- added USB1: USB_C_Receptacle_USB2.0_14P, Connector_USB:USB_C_Receptacle_HRO_TYPE-C-31-M-12, F.Cu at (-124.2, 120.8)

Commit message: Tarea 3
Parts:
- moved USB1 279.3 mm to (146.0, 50.0), turned to 90 degrees
- moved Q8 275.2 mm to (126.6, 48.3), turned to 180 degrees
- moved OC14 267.3 mm to (133.0, 53.0), turned to 90 degrees
- moved R2 267.0 mm to (140.0, 45.5), turned to 90 degrees
- moved R66 265.7 mm to (140.0, 54.0), turned to 180 degrees
- moved R1 264.2 mm to (140.0, 55.0), turned to 180 degrees
- moved D22 262.1 mm to (138.5, 48.0)
- moved D12 252.7 mm to (129.0, 57.5), turned to 90 degrees
- moved D18 251.6 mm to (139.5, 51.5), turned to -90 degrees
- moved R48 244.7 mm to (134.5, 46.0)
- moved R50 242.4 mm to (131.0, 46.0), turned to 180 degrees
- moved R59 238.6 mm to (129.0, 54.0), turned to 90 degrees
- moved R45 235.7 mm to (131.0, 61.0)
- moved L1 194.6 mm to (141.5, 102.5), turned to -90 degrees
- moved K2 190.0 mm to (90.4, 47.7), turned to 180 degrees
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
Commit message: Tarea 3
Parts:
- moved Q1 287.9 mm to (156.1, 55.8), turned to 180 degrees
- moved D3 275.3 mm to (161.5, 62.5), turned to 90 degrees
- moved R24 270.4 mm to (160.5, 57.5), turned to 90 degrees
- moved Q3 268.3 mm to (141.3, 89.9), turned to -90 degrees
- moved R23 263.8 mm to (155.5, 60.5), turned to 180 degrees
- moved R20 258.3 mm to (150.5, 60.0), turned to 90 degrees
- moved R19 255.9 mm to (153.0, 73.0)
- moved R25 255.4 mm to (160.5, 88.0), turned to -90 degrees
- moved D4 253.4 mm to (146.0, 88.0), turned to 90 degrees
- moved R26 249.7 mm to (155.5, 94.5)
- moved R27 241.8 mm to (146.0, 91.5), turned to 90 degrees
- moved R28 241.3 mm to (143.5, 86.5), turned to 180 degrees
- moved Q2 238.0 mm to (113.4, 95.2)
- moved OC10 225.9 mm to (152.5, 102.0), turned to 0 degrees
- moved R9 225.8 mm to (124.0, 97.5)
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
Commit message: tarea 3 - update
Parts:
- removed C7: 10uF, PCM_Capacitor_SMD_AKL:C_0603_1608Metric
- removed D1: SMBJ12CA, PCM_Diode_SMD_AKL:D_SMB_TVS
- removed D16: SMAJ5.0A, PCM_Diode_SMD_AKL:D_SMA
- removed D8: SM712, PCM_Package_TO_SOT_SMD_AKL:SOT-23
- removed R39, R40: 47K, PCM_Resistor_SMD_AKL:R_0603_1608Metric
- added J4: Conn_01x03, Connector_PinHeader_2.54mm:PinHeader_1x03_P2.54mm_Vertical, F.Cu at (131.5, 64.5)
- added REF**: MountingHole_2.2mm_M2, MountingHole:MountingHole_2.2mm_M2, F.Cu at (153.5, 49.0)
- added REF**: MountingHole_2.2mm_M2, MountingHole:MountingHole_2.2mm_M2, F.Cu at (73.0, 100.5)
- added U21: ~, rs485_footprint:SOIC127P600X175-8N, F.Cu at (144.5, 63.5)
- moved R56 20.6 mm to (116.0, 81.5), turned to 180 degrees
- moved R48 14.8 mm to (121.5, 54.0), turned to 180 degrees
- moved R21 14.6 mm to (85.5, 103.0)
- moved R11 10.5 mm to (78.3, 103.0)
- moved C12 9.71 mm to (147.5, 70.5), turned to 0 degrees
- moved R12 9.00 mm to (135.5, 84.0)
- moved R8 8.14 mm to (148.5, 68.5), turned to 0 degrees
- moved R45 7.63 mm to (121.0, 67.5)
- moved R7 7.50 mm to (124.5, 67.5), turned to 0 degrees
- moved R13 6.40 mm to (140.5, 86.5), turned to 180 degrees
- moved D19 6.02 mm to (153.5, 66.5)
- moved D12 5.66 mm to (125.0, 54.5), turned to 180 degrees
- moved R22 5.32 mm to (82.5, 99.0)
- moved C5 4.96 mm to (85.4, 88.5)
- moved R20 4.74 mm to (155.0, 61.5)
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Routing:
- net GND: track 0.00 -> 350.5 mm
- net VCC: track 0.00 -> 145.2 mm
- net /Board-PLC4UNI-G1w/4_NPN_OUT: track 0.00 -> 66.9 mm
- net Net-(D9-A): track 0.00 -> 48.1 mm
- net +3.3V: track 0.00 -> 37.0 mm
- net /Board-PLC4UNI-G1w/NO_A_RLY: track 0.00 -> 36.1 mm
- net /Board-PLC4UNI-G1w/COM_A_RLY: track 0.00 -> 33.5 mm
- net /Board-PLC4UNI-G1w/2_PNP_IN: track 0.00 -> 31.5 mm
- net Net-(D10-A): track 0.00 -> 25.7 mm
- net (no net): track 0.00 -> 21.4 mm
- net /Board-PLC4UNI-G1w/COM_B_RLY: track 0.00 -> 21.1 mm
- net /Board-PLC4UNI-G1w/NO_B_RLY: track 0.00 -> 20.0 mm
- net Net-(D17-A): track 0.00 -> 14.8 mm
- net /Board-PLC4UNI-G1w/2_NPN_IN: track 0.00 -> 12.1 mm
- net Net-(Q1-B): track 0.00 -> 10.8 mm
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Other:
- board outline added: 100.1 x 80.2 mm

Commit message: Tarea 3 - Update
Parts:
- C13: footprint PCM_Capacitor_SMD_AKL:C_0603_1608Metric -> Capacitor_SMD:C_0805_2012Metric_Pad1.18x1.45mm_HandSolder
Routing:
- net VCC: track 145.2 -> 335.8 mm, vias 0 -> 19
- net GND: track 350.5 -> 504.5 mm, vias 0 -> 33
- net /Board-PLC4UNI-G1w/4-20mA_Input: track 1.76 -> 150.7 mm, vias 0 -> 6
- net /Board-PLC4UNI-G1w/PLC4UNI_CPU/FROMESP_IN_OUT-NPN_C: track 0.00 -> 140.5 mm, vias 0 -> 4
- net +3.3V: track 37.0 -> 170.4 mm, vias 0 -> 14
- net /Board-PLC4UNI-G1w/4-20mA_Input/4-20mA_toESP_IN: track 3.71 -> 125.4 mm, vias 0 -> 8
- net /Board-PLC4UNI-G1w/3_NPN_OUT: track 3.98 -> 102.1 mm, vias 0 -> 1
- net /Board-PLC4UNI-G1w/2_NPN_OUT: track 4.11 -> 101.3 mm, vias 0 -> 1
- net /Board-PLC4UNI-G1w/PLC4UNI_CPU/FROMESP_IN_OUT-PNP_B: track 0.00 -> 87.0 mm, vias 0 -> 2
- net /Board-PLC4UNI-G1w/2_PNP_OUT: track 5.42 -> 84.7 mm, vias 0 -> 2
- net /Board-PLC4UNI-G1w/PLC4UNI_CPU/USB-: track 0.00 -> 76.5 mm, vias 0 -> 10
- net /Board-PLC4UNI-G1w/PLC4UNI_CPU/ESP32_UART_B: track 0.00 -> 76.3 mm, vias 0 -> 6
- net /Board-PLC4UNI-G1w/PLC4UNI_CPU/FROMESP_OUT_IN-PNP_B: track 2.46 -> 77.7 mm, vias 0 -> 6
- net /Board-PLC4UNI-G1w/PLC4UNI_CPU/USB+: track 0.00 -> 75.2 mm, vias 0 -> 9
- net /Board-PLC4UNI-G1w/1_NPN_OUT: track 0.00 -> 73.3 mm, vias 0 -> 1
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