File: Tarea 3/Diseño PCB/PLC4UNI/4-20mA_Output.kicad_sch (KiCad schematic)
At the start: 13 parts, among them Q10 IRLML6402TRPBF-JSM, U3 GP8303-TC50-EW

Commit message: Tarea 3
Connections:
- no-connect marks 0 -> 4
Changed lines of the file:
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@@
 		(color 0 0 0 0)
+	)
+	(no_connect
+		(at 111.76 73.66)
+	)
+	(no_connect
+		(at 111.76 76.2)
+	)
+	(no_connect
+		(at 91.44 78.74)
+	)
+	(no_connect
+		(at 91.44 81.28)
 	)
 	(wire

Commit message: Tarea - Update
Parts:
- C13: footprint PCM_Capacitor_SMD_AKL:C_0603_1608Metric -> Capacitor_SMD:C_0805_2012Metric_Pad1.18x1.45mm_HandSolder
Changed lines of the file:
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@@
 			)
 		)
-		(property "Footprint" "PCM_Capacitor_SMD_AKL:C_0603_1608Metric"
+		(property "Footprint" "Capacitor_SMD:C_0805_2012Metric_Pad1.18x1.45mm_HandSolder"
 			(at 132.3848 91.44 0)
 			(effects
